Commit message: add encoders estimation

File: ws/src/four_ws_vehicle_simulation/models/wheeled_robot.urdf (robot description, URDF)
Before this commit: robot wheeled_robot, 8 links, 7 joints
Links:
- link back_left_wheel: mass 2 -> 0.2
- link back_right_wheel: mass 2 -> 0.2
- link front_left_wheel: mass 2 -> 0.2
- link front_left_wheel_steering: mass 2 -> 0.2
- link front_right_wheel: mass 2 -> 0.2
- link front_right_wheel_steering: mass 2 -> 0.2
